Commit message: Added changes from devel/actions to master

File: robot_models/urdf_models/robot_setups/kuka_iiwa/use_case_setup_iiwa.urdf (robot description, URDF)
Before this commit: robot iiwa_setup, 14 links, 13 joints
Joints:
- joint right_ft_sensor_joint: origin xyz=0 0 0.0225 rpy=0 3.1416 -0.7854 -> xyz=0 0 0.0225 rpy=0 0 3.1416

File: robot_models/urdf_models/robot_setups/kuka_iiwa/use_case_setup_iiwa.urdf.xacro (robot description, xacro)
@@ -50,5 +50,5 @@
   <link name="${prefix_right}ft_sensor_frame"/>
   	<joint name="${prefix_right}ft_sensor_joint" type="fixed">
-  		<origin xyz="0 0 ${0.01 + 0.025/2}" rpy="${0} ${3.1416} ${-3.1416/4}"/>
+  		<origin xyz="0 0 ${0.01 + 0.025/2}" rpy="${0} ${0} ${3.1416}"/>
   		<parent link="${prefix_right}tool0"/>
   		<child link="${prefix_right}ft_sensor_frame"/>
