Commit message: Calibration working

File: robot_models/urdf_models/robot_setups/neura_maira7M/use_case_setup_neura_maira7M.urdf.xacro (robot description, xacro)
@@ -10,7 +10,13 @@
 	<link name="world" />
 	<joint name="world_joint" type="fixed">
-	<parent link="world" />
-	<child link = "$(arg prefix)root_link" />
-	<origin xyz="0.0 0.0 0.0" rpy="0.0 0.0 0.0" />
+		<parent link="world" />
+		<child link = "$(arg prefix)root_link" />
+		<origin xyz="0.0 0.0 0.0" rpy="0.0 0.0 0.0" />
+	</joint>
+	<link name="FT_sensor_frame" />
+	<joint name="FT_sensor_frame_joint" type="fixed">
+		<parent link="FT_sensor_frame" />
+		<child link = "$(arg prefix)root_link" />
+		<origin xyz="0.0 0.0 0.0" rpy="0.0 0.0 0.0" />
 	</joint>
 </robot>
