Commit message: Neura robot running properly

File: robot_models/urdf_models/robot_setups/neura_maira7M/use_case_setup_neura_maira7M.urdf (robot description, URDF)
Before this commit: robot robelix_neura_robot, 11 links, 10 joints
Joints:
- joint maira7M_joint7: limit lower=-3.14159 upper=3.14159 effort=37 velocity=3.14159 -> lower=-3.0 upper=3.0 effort=37 velocity=1.57

Commit message: Added ft sensor frame to the urdf of maira

File: robot_models/urdf_models/robot_setups/neura_maira7M/use_case_setup_neura_maira7M.urdf (robot description, URDF)
Before this commit: robot robelix_neura_robot, 11 links, 10 joints
Links:
- added link FT_sensor_frame
Joints:
- added joint FT_sensor_frame_joint: type fixed, parent FT_sensor_frame, child maira7M_flange, origin xyz=0.0 0.0 0.0 rpy=0.0 0.0 0.0
- joint maira7M_joint7: limit lower=-3.0 upper=3.0 effort=37 velocity=1.57 -> lower=-3.14159 upper=3.14159 effort=37 velocity=3.14159

File: robot_models/urdf_models/robot_setups/neura_maira7M/use_case_setup_neura_maira7M.urdf.xacro (robot description, xacro)
@@ -17,5 +17,5 @@
 	<joint name="FT_sensor_frame_joint" type="fixed">
 		<parent link="FT_sensor_frame" />
-		<child link = "$(arg prefix)root_link" />
+		<child link = "$(arg prefix)flange" />
 		<origin xyz="0.0 0.0 0.0" rpy="0.0 0.0 0.0" />
 	</joint>

Commit message: Fix ft sensor transform

File: robot_models/urdf_models/robot_setups/neura_maira7M/use_case_setup_neura_maira7M.urdf (robot description, URDF)
Before this commit: robot robelix_neura_robot, 12 links, 11 joints
Joints:
- joint FT_sensor_frame_joint: child maira7M_flange -> FT_sensor_frame; parent FT_sensor_frame -> maira7M_flange

File: robot_models/urdf_models/robot_setups/neura_maira7M/use_case_setup_neura_maira7M.urdf.xacro (robot description, xacro)
@@ -16,6 +16,6 @@
 	<link name="FT_sensor_frame" />
 	<joint name="FT_sensor_frame_joint" type="fixed">
-		<parent link="FT_sensor_frame" />
-		<child link = "$(arg prefix)flange" />
+		<parent link="$(arg prefix)flange" />
+		<child link = "FT_sensor_frame" />
 		<origin xyz="0.0 0.0 0.0" rpy="0.0 0.0 0.0" />
 	</joint>

Commit message: Fix ft sensor transform

File: robot_models/urdf_models/robot_setups/neura_maira7M/use_case_setup_neura_maira7M.urdf (robot description, URDF)
Before this commit: robot robelix_neura_robot, 12 links, 11 joints
Joints:
- joint FT_sensor_frame_joint: origin xyz=0.0 0.0 0.0 rpy=0.0 0.0 0.0 -> xyz=0.0 0.0 0.066 rpy=0.0 0.0 0.0
- joint maira7M_link7_to_flange: origin xyz=0 0.115 0 rpy=-1.5707963267948966 -1.5707963267948966 0 -> xyz=0 0.135 0 rpy=-1.5707963267948966 -1.5707963267948966 0

File: robot_models/urdf_models/robot_setups/neura_maira7M/use_case_setup_neura_maira7M.urdf.xacro (robot description, xacro)
@@ -18,5 +18,5 @@
 		<parent link="$(arg prefix)flange" />
 		<child link = "FT_sensor_frame" />
-		<origin xyz="0.0 0.0 0.0" rpy="0.0 0.0 0.0" />
+		<origin xyz="0.0 0.0 0.066" rpy="0.0 0.0 0.0" />
 	</joint>
 </robot>
