Commit message: Implemented kinematic constraints of robelix robot model (differential drive). Also implemented fixturefor only move when outside of a sphere. All this is implemented at the robot model side and not at the task specification side

File: robot_models/urdf_models/robot_setups/robelix/use_case_setup_robelix_mobile.urdf (robot description, URDF)
Before this commit: robot robelix_neura_robot, 36 links, 35 joints
Joints:
- joint theta_mobile_joint: limit lower=-30 upper=30 effort=100000 velocity=0.51 -> lower=-30 upper=30 effort=100000 velocity=0.3
- joint x_mobile_joint: limit lower=-100 upper=100 effort=100000 velocity=0.5 -> lower=-100 upper=100 effort=100000 velocity=0.2
- joint y_mobile_joint: limit lower=-100 upper=100 effort=100000 velocity=0.5 -> lower=-100 upper=100 effort=100000 velocity=0.2

File: robot_models/urdf_models/robot_setups/robelix/use_case_setup_robelix_mobile.urdf.xacro (robot description, xacro)
@@ -25,5 +25,5 @@
                 <child link="x_mobile_link" />
                 <axis xyz="1 0 0" />
-                <limit lower="-100" upper="100" effort="100000" velocity="0.5" />
+                <limit lower="-100" upper="100" effort="100000" velocity="0.2" />
         </joint>
         <link name="y_mobile_link" />
@@ -33,5 +33,5 @@
                 <child link="y_mobile_link" />
                 <axis xyz="0 1 0" />
-                <limit lower="-100" upper="100" effort="100000" velocity="0.5" />
+                <limit lower="-100" upper="100" effort="100000" velocity="0.2" />
         </joint>
         <!-- TODO: change the following to continous when Erwin enables that type of joint in the urdf reader -->
@@ -41,5 +41,5 @@
                 <child link="$(arg robot_ns)_base_link" />
                 <axis xyz="0 0 1" />
-                <limit lower="-30" upper="30" effort="100000" velocity="0.51" />
+                <limit lower="-30" upper="30" effort="100000" velocity="0.3" />
 	    </joint>
 	</xacro:unless>

Commit message: MAV alignment and jointspace with Maira, insertions working, and extra testing skills

File: robot_models/urdf_models/robot_setups/robelix/use_case_setup_robelix_mobile.urdf (robot description, URDF)
Before this commit: robot robelix_neura_robot, 39 links, 38 joints
Links:
- added link tool0_grip_rot
- added link tool0_insertions
Joints:
- added joint tool0_grip_rot_joint: type fixed, parent tool0_grip, child tool0_grip_rot, origin xyz=0.0 0.0 0.0 rpy=0.0 -1.0472 0.0
- added joint tool0_insertions_joint: type fixed, parent tool0_grip_rot, child tool0_insertions, origin xyz=0.0 0.0 -0.085 rpy=0.0 0.0 -1.5708
- joint theta_mobile_joint: limit lower=-30 upper=30 effort=100000 velocity=0.3 -> lower=-30 upper=30 effort=100000 velocity=0.15

File: robot_models/urdf_models/robot_setups/robelix/use_case_setup_robelix_mobile.urdf.xacro (robot description, xacro)
@@ -41,5 +41,5 @@
                 <child link="$(arg robot_ns)_base_link" />
                 <axis xyz="0 0 1" />
-                <limit lower="-30" upper="30" effort="100000" velocity="0.3" />
+                <limit lower="-30" upper="30" effort="100000" velocity="0.15" />
 	    </joint>
 	</xacro:unless>
@@ -56,4 +56,16 @@
 		<origin xyz="0.0 0.0 0.18" rpy="0.0 3.1416 0.0" />
 	</joint>
+    <link name="tool0_grip_rot" />
+	<joint name="tool0_grip_rot_joint" type="fixed">
+		<parent link="tool0_grip" />
+		<child link = "tool0_grip_rot" />
+		<origin xyz="0.0 0.0 0.0" rpy="0.0 -1.0472 0.0" />
+	</joint>
+    <link name="tool0_insertions" />
+	<joint name="tool0_insertions_joint" type="fixed">
+		<parent link="tool0_grip_rot" />
+		<child link = "tool0_insertions" />
+		<origin xyz="0.0 0.0 -0.085" rpy="0.0 0.0 -1.5708" />
+	</joint>
     <link name="tool0_cables" />
 	<joint name="tool0_cables_joint" type="fixed">
