Commit message: Added ft sensor frame to urdfs with mav

File: robot_models/urdf_models/robot_setups/robelix/use_case_setup_robelix_fixed.urdf (robot description, URDF)
Before this commit: robot robelix_neura_robot, 34 links, 33 joints
Links:
- added link FT_sensor_frame
Joints:
- added joint FT_sensor_frame_joint: type fixed, parent maira7M_flange, child FT_sensor_frame, origin xyz=0.0 0.0 0.066 rpy=0.0 0.0 0.0
- joint maira7M_link7_to_flange: origin xyz=0 0.115 0 rpy=-1.5707963267948966 -1.5707963267948966 0 -> xyz=0 0.135 0 rpy=-1.5707963267948966 -1.5707963267948966 0

File: robot_models/urdf_models/robot_setups/robelix/use_case_setup_robelix_fixed.urdf.xacro (robot description, xacro)
@@ -15,3 +15,9 @@
         <origin xyz="$(arg tx) $(arg ty) $(arg tz)" rpy="$(arg rr) $(arg rp) $(arg ry)" />
     </joint>
+    <link name="FT_sensor_frame" />
+	<joint name="FT_sensor_frame_joint" type="fixed">
+		<parent link="$(arg prefix)flange" />
+		<child link = "FT_sensor_frame" />
+		<origin xyz="0.0 0.0 0.066" rpy="0.0 0.0 0.0" />
+	</joint>
 </robot>

File: robot_models/urdf_models/robot_setups/robelix/use_case_setup_robelix_mobile.urdf (robot description, URDF)
Before this commit: robot robelix_neura_robot, 36 links, 35 joints
Links:
- added link FT_sensor_frame
Joints:
- added joint FT_sensor_frame_joint: type fixed, parent maira7M_flange, child FT_sensor_frame, origin xyz=0.0 0.0 0.066 rpy=0.0 0.0 0.0
- joint maira7M_link7_to_flange: origin xyz=0 0.115 0 rpy=-1.5707963267948966 -1.5707963267948966 0 -> xyz=0 0.135 0 rpy=-1.5707963267948966 -1.5707963267948966 0

File: robot_models/urdf_models/robot_setups/robelix/use_case_setup_robelix_mobile.urdf.xacro (robot description, xacro)
@@ -44,3 +44,9 @@
 	    </joint>
 	</xacro:unless>
+    <link name="FT_sensor_frame" />
+	<joint name="FT_sensor_frame_joint" type="fixed">
+		<parent link="$(arg prefix)flange" />
+		<child link = "FT_sensor_frame" />
+		<origin xyz="0.0 0.0 0.066" rpy="0.0 0.0 0.0" />
+	</joint>
 </robot>

Commit message: Fixed yaw of robot base link

File: robot_models/urdf_models/robot_setups/robelix/use_case_setup_robelix_fixed.urdf (robot description, URDF)
Before this commit: robot robelix_neura_robot, 35 links, 34 joints
Joints:
- joint robot_base_flange: origin xyz=0 0 0 rpy=0 0 3.141592653589793 -> xyz=0 0 0 rpy=0 0 1.5708026535897932

File: robot_models/urdf_models/robot_setups/robelix/use_case_setup_robelix_fixed.urdf.xacro (robot description, xacro)
@@ -7,5 +7,5 @@
 	<xacro:mav_plus axes_config="fixed" gripper="" arm_name="maira7M"
             backpack="" lin_axis_base_x="0.52" lin_axis_base_z="0.8125" lin_axis_height="0.345"
-            robot_base_yaw="0.0" camera_setup="link6" complex_mav_urdf="true" fixed_wheels="true"
+            robot_base_yaw="-1.57079" camera_setup="link6" complex_mav_urdf="true" fixed_wheels="true"
             klt_box="false" small_klt_box="false"/>
 	<link name="world" />

File: robot_models/urdf_models/robot_setups/robelix/use_case_setup_robelix_mobile.urdf (robot description, URDF)
Before this commit: robot robelix_neura_robot, 37 links, 36 joints
Joints:
- joint robot_base_flange: origin xyz=0 0 0 rpy=0 0 3.141592653589793 -> xyz=0 0 0 rpy=0 0 1.5708026535897932

File: robot_models/urdf_models/robot_setups/robelix/use_case_setup_robelix_mobile.urdf.xacro (robot description, xacro)
@@ -8,5 +8,5 @@
 	<xacro:mav_plus axes_config="fixed" gripper="" arm_name="maira7M"
             backpack="" lin_axis_base_x="0.52" lin_axis_base_z="0.8125" lin_axis_height="0.345"
-            robot_base_yaw="0.0" camera_setup="link6" complex_mav_urdf="true" fixed_wheels="true"
+            robot_base_yaw="-1.57079" camera_setup="link6" complex_mav_urdf="true" fixed_wheels="true"
             klt_box="false" small_klt_box="false"/>
 	<link name="world" />

Commit message: Fixed yaw of robot base link

File: robot_models/urdf_models/robot_setups/robelix/use_case_setup_robelix_fixed.urdf (robot description, URDF)
Before this commit: robot robelix_neura_robot, 35 links, 34 joints
Joints:
- joint robot_base_flange: origin xyz=0 0 0 rpy=0 0 1.5708026535897932 -> xyz=0 0 0 rpy=0 0 2.3561946535897933

File: robot_models/urdf_models/robot_setups/robelix/use_case_setup_robelix_fixed.urdf.xacro (robot description, xacro)
@@ -7,5 +7,5 @@
 	<xacro:mav_plus axes_config="fixed" gripper="" arm_name="maira7M"
             backpack="" lin_axis_base_x="0.52" lin_axis_base_z="0.8125" lin_axis_height="0.345"
-            robot_base_yaw="-1.57079" camera_setup="link6" complex_mav_urdf="true" fixed_wheels="true"
+            robot_base_yaw="-0.785398" camera_setup="link6" complex_mav_urdf="true" fixed_wheels="true"
             klt_box="false" small_klt_box="false"/>
 	<link name="world" />

File: robot_models/urdf_models/robot_setups/robelix/use_case_setup_robelix_mobile.urdf (robot description, URDF)
Before this commit: robot robelix_neura_robot, 37 links, 36 joints
Joints:
- joint robot_base_flange: origin xyz=0 0 0 rpy=0 0 1.5708026535897932 -> xyz=0 0 0 rpy=0 0 2.3561946535897933

File: robot_models/urdf_models/robot_setups/robelix/use_case_setup_robelix_mobile.urdf.xacro (robot description, xacro)
@@ -8,5 +8,5 @@
 	<xacro:mav_plus axes_config="fixed" gripper="" arm_name="maira7M"
             backpack="" lin_axis_base_x="0.52" lin_axis_base_z="0.8125" lin_axis_height="0.345"
-            robot_base_yaw="-1.57079" camera_setup="link6" complex_mav_urdf="true" fixed_wheels="true"
+            robot_base_yaw="-0.785398" camera_setup="link6" complex_mav_urdf="true" fixed_wheels="true"
             klt_box="false" small_klt_box="false"/>
 	<link name="world" />

Commit message: Added tcps tool0_cables and tool0_grip links

File: robot_models/urdf_models/robot_setups/robelix/use_case_setup_robelix_fixed.urdf (robot description, URDF)
Before this commit: robot robelix_neura_robot, 35 links, 34 joints
Links:
- added link tool0_cables
- added link tool0_grip
Joints:
- added joint tool0_cables_joint: type fixed, parent FT_sensor_frame, child tool0_cables, origin xyz=0.0 0.0 0.14 rpy=0.0 0.0 0.0
- added joint tool0_grip_joint: type fixed, parent FT_sensor_frame, child tool0_grip, origin xyz=0.0 0.0 0.18 rpy=0.0 0.0 0.0

File: robot_models/urdf_models/robot_setups/robelix/use_case_setup_robelix_fixed.urdf.xacro (robot description, xacro)
@@ -21,3 +21,15 @@
 		<origin xyz="0.0 0.0 0.066" rpy="0.0 0.0 0.0" />
 	</joint>
+    <link name="tool0_grip" />
+	<joint name="tool0_grip_joint" type="fixed">
+		<parent link="FT_sensor_frame" />
+		<child link = "tool0_grip" />
+		<origin xyz="0.0 0.0 0.18" rpy="0.0 0.0 0.0" />
+	</joint>
+    <link name="tool0_cables" />
+	<joint name="tool0_cables_joint" type="fixed">
+		<parent link="FT_sensor_frame" />
+		<child link = "tool0_cables" />
+		<origin xyz="0.0 0.0 0.14" rpy="0.0 0.0 0.0" />
+	</joint>
 </robot>

File: robot_models/urdf_models/robot_setups/robelix/use_case_setup_robelix_mobile.urdf (robot description, URDF)
Before this commit: robot robelix_neura_robot, 37 links, 36 joints
Links:
- added link tool0_cables
- added link tool0_grip
Joints:
- added joint tool0_cables_joint: type fixed, parent FT_sensor_frame, child tool0_cables, origin xyz=0.0 0.0 0.14 rpy=0.0 0.0 0.0
- added joint tool0_grip_joint: type fixed, parent FT_sensor_frame, child tool0_grip, origin xyz=0.0 0.0 0.18 rpy=0.0 0.0 0.0

File: robot_models/urdf_models/robot_setups/robelix/use_case_setup_robelix_mobile.urdf.xacro (robot description, xacro)
@@ -50,3 +50,15 @@
 		<origin xyz="0.0 0.0 0.066" rpy="0.0 0.0 0.0" />
 	</joint>
+    <link name="tool0_grip" />
+	<joint name="tool0_grip_joint" type="fixed">
+		<parent link="FT_sensor_frame" />
+		<child link = "tool0_grip" />
+		<origin xyz="0.0 0.0 0.18" rpy="0.0 0.0 0.0" />
+	</joint>
+    <link name="tool0_cables" />
+	<joint name="tool0_cables_joint" type="fixed">
+		<parent link="FT_sensor_frame" />
+		<child link = "tool0_cables" />
+		<origin xyz="0.0 0.0 0.14" rpy="0.0 0.0 0.0" />
+	</joint>
 </robot>

Commit message: Rotated tool tcp for cables

File: robot_models/urdf_models/robot_setups/robelix/use_case_setup_robelix_fixed.urdf (robot description, URDF)
Before this commit: robot robelix_neura_robot, 37 links, 36 joints
Joints:
- joint tool0_cables_joint: origin xyz=0.0 0.0 0.14 rpy=0.0 0.0 0.0 -> xyz=0.0 0.0 0.14 rpy=0.0 3.1416 0.0

File: robot_models/urdf_models/robot_setups/robelix/use_case_setup_robelix_fixed.urdf.xacro (robot description, xacro)
@@ -31,5 +31,5 @@
 		<parent link="FT_sensor_frame" />
 		<child link = "tool0_cables" />
-		<origin xyz="0.0 0.0 0.14" rpy="0.0 0.0 0.0" />
+		<origin xyz="0.0 0.0 0.14" rpy="0.0 3.1416 0.0" />
 	</joint>
 </robot>

File: robot_models/urdf_models/robot_setups/robelix/use_case_setup_robelix_mobile.urdf (robot description, URDF)
Before this commit: robot robelix_neura_robot, 39 links, 38 joints
Joints:
- joint tool0_cables_joint: origin xyz=0.0 0.0 0.14 rpy=0.0 0.0 0.0 -> xyz=0.0 0.0 0.14 rpy=0.0 3.1416 0.0

File: robot_models/urdf_models/robot_setups/robelix/use_case_setup_robelix_mobile.urdf.xacro (robot description, xacro)
@@ -60,5 +60,5 @@
 		<parent link="FT_sensor_frame" />
 		<child link = "tool0_cables" />
-		<origin xyz="0.0 0.0 0.14" rpy="0.0 0.0 0.0" />
+		<origin xyz="0.0 0.0 0.14" rpy="0.0 3.1416 0.0" />
 	</joint>
 </robot>

Commit message: Updated frames for tcp

File: robot_models/urdf_models/robot_setups/robelix/use_case_setup_robelix_fixed.urdf (robot description, URDF)
Before this commit: robot robelix_neura_robot, 37 links, 36 joints
Links:
- added link tool0_cables_intermediate
Joints:
- added joint tool0_cables_intermediate_joint: type fixed, parent FT_sensor_frame, child tool0_cables_intermediate, origin xyz=0.0 0.0 0.14 rpy=0.0 3.1416 0.0
- joint tool0_cables_joint: origin xyz=0.0 0.0 0.14 rpy=0.0 3.1416 0.0 -> xyz=0.0 0.0 0.0 rpy=0.0 0.0 0.785398; parent FT_sensor_frame -> tool0_cables_intermediate

File: robot_models/urdf_models/robot_setups/robelix/use_case_setup_robelix_fixed.urdf.xacro (robot description, xacro)
@@ -27,9 +27,15 @@
 		<origin xyz="0.0 0.0 0.18" rpy="0.0 0.0 0.0" />
 	</joint>
+    <link name="tool0_cables_intermediate" />
+	<joint name="tool0_cables_intermediate_joint" type="fixed">
+		<parent link="FT_sensor_frame" />
+		<child link = "tool0_cables_intermediate" />
+		<origin xyz="0.0 0.0 0.14" rpy="0.0 3.1416 0.0" />
+	</joint>
     <link name="tool0_cables" />
 	<joint name="tool0_cables_joint" type="fixed">
-		<parent link="FT_sensor_frame" />
+		<parent link="tool0_cables_intermediate" />
 		<child link = "tool0_cables" />
-		<origin xyz="0.0 0.0 0.14" rpy="0.0 3.1416 0.0" />
+		<origin xyz="0.0 0.0 0.0" rpy="0.0 0.0 0.785398" />
 	</joint>
 </robot>

File: robot_models/urdf_models/robot_setups/robelix/use_case_setup_robelix_mobile.urdf (robot description, URDF)
Before this commit: robot robelix_neura_robot, 39 links, 38 joints
Links:
- added link tool0_cables_intermediate
Joints:
- added joint tool0_cables_intermediate_joint: type fixed, parent FT_sensor_frame, child tool0_cables_intermediate, origin xyz=0.0 0.0 0.14 rpy=0.0 3.1416 0.0
- joint tool0_cables_joint: origin xyz=0.0 0.0 0.14 rpy=0.0 3.1416 0.0 -> xyz=0.0 0.0 0.0 rpy=0.0 0.0 0.785398; parent FT_sensor_frame -> tool0_cables_intermediate

File: robot_models/urdf_models/robot_setups/robelix/use_case_setup_robelix_mobile.urdf.xacro (robot description, xacro)
@@ -56,9 +56,15 @@
 		<origin xyz="0.0 0.0 0.18" rpy="0.0 0.0 0.0" />
 	</joint>
+    <link name="tool0_cables_intermediate" />
+	<joint name="tool0_cables_intermediate_joint" type="fixed">
+		<parent link="FT_sensor_frame" />
+		<child link = "tool0_cables_intermediate" />
+		<origin xyz="0.0 0.0 0.14" rpy="0.0 3.1416 0.0" />
+	</joint>
     <link name="tool0_cables" />
 	<joint name="tool0_cables_joint" type="fixed">
-		<parent link="FT_sensor_frame" />
+		<parent link="tool0_cables_intermediate" />
 		<child link = "tool0_cables" />
-		<origin xyz="0.0 0.0 0.14" rpy="0.0 3.1416 0.0" />
+		<origin xyz="0.0 0.0 0.0" rpy="0.0 0.0 0.785398" />
 	</joint>
 </robot>

Commit message: Updated frames for tcp

File: robot_models/urdf_models/robot_setups/robelix/use_case_setup_robelix_fixed.urdf (robot description, URDF)
Before this commit: robot robelix_neura_robot, 38 links, 37 joints
Joints:
- joint tool0_cables_joint: origin xyz=0.0 0.0 0.0 rpy=0.0 0.0 0.785398 -> xyz=0.0 0.0 0.0 rpy=0.0 0.0 -0.785398

File: robot_models/urdf_models/robot_setups/robelix/use_case_setup_robelix_fixed.urdf.xacro (robot description, xacro)
@@ -37,5 +37,5 @@
 		<parent link="tool0_cables_intermediate" />
 		<child link = "tool0_cables" />
-		<origin xyz="0.0 0.0 0.0" rpy="0.0 0.0 0.785398" />
+		<origin xyz="0.0 0.0 0.0" rpy="0.0 0.0 -0.785398" />
 	</joint>
 </robot>

File: robot_models/urdf_models/robot_setups/robelix/use_case_setup_robelix_mobile.urdf (robot description, URDF)
Before this commit: robot robelix_neura_robot, 40 links, 39 joints
Joints:
- joint tool0_cables_joint: origin xyz=0.0 0.0 0.0 rpy=0.0 0.0 0.785398 -> xyz=0.0 0.0 0.0 rpy=0.0 0.0 -0.785398

File: robot_models/urdf_models/robot_setups/robelix/use_case_setup_robelix_mobile.urdf.xacro (robot description, xacro)
@@ -66,5 +66,5 @@
 		<parent link="tool0_cables_intermediate" />
 		<child link = "tool0_cables" />
-		<origin xyz="0.0 0.0 0.0" rpy="0.0 0.0 0.785398" />
+		<origin xyz="0.0 0.0 0.0" rpy="0.0 0.0 -0.785398" />
 	</joint>
 </robot>

Commit message: Updated frames for tcp

File: robot_models/urdf_models/robot_setups/robelix/use_case_setup_robelix_fixed.urdf (robot description, URDF)
Before this commit: robot robelix_neura_robot, 38 links, 37 joints
Links:
- removed link tool0_cables_intermediate
Joints:
- removed joint tool0_cables_intermediate_joint
- joint tool0_cables_joint: origin xyz=0.0 0.0 0.0 rpy=0.0 0.0 -0.785398 -> xyz=0.0 0.0 0.14 rpy=0.0 3.1416 0.0; parent tool0_cables_intermediate -> FT_sensor_frame

File: robot_models/urdf_models/robot_setups/robelix/use_case_setup_robelix_fixed.urdf.xacro (robot description, xacro)
@@ -27,15 +27,9 @@
 		<origin xyz="0.0 0.0 0.18" rpy="0.0 0.0 0.0" />
 	</joint>
-    <link name="tool0_cables_intermediate" />
-	<joint name="tool0_cables_intermediate_joint" type="fixed">
+    <link name="tool0_cables" />
+	<joint name="tool0_cables_joint" type="fixed">
 		<parent link="FT_sensor_frame" />
-		<child link = "tool0_cables_intermediate" />
+		<child link = "tool0_cables" />
 		<origin xyz="0.0 0.0 0.14" rpy="0.0 3.1416 0.0" />
 	</joint>
-    <link name="tool0_cables" />
-	<joint name="tool0_cables_joint" type="fixed">
-		<parent link="tool0_cables_intermediate" />
-		<child link = "tool0_cables" />
-		<origin xyz="0.0 0.0 0.0" rpy="0.0 0.0 -0.785398" />
-	</joint>
 </robot>

File: robot_models/urdf_models/robot_setups/robelix/use_case_setup_robelix_mobile.urdf (robot description, URDF)
Before this commit: robot robelix_neura_robot, 40 links, 39 joints
Links:
- removed link tool0_cables_intermediate
Joints:
- removed joint tool0_cables_intermediate_joint
- joint tool0_cables_joint: origin xyz=0.0 0.0 0.0 rpy=0.0 0.0 -0.785398 -> xyz=0.0 0.0 0.14 rpy=0.0 3.1416 0.0; parent tool0_cables_intermediate -> FT_sensor_frame

File: robot_models/urdf_models/robot_setups/robelix/use_case_setup_robelix_mobile.urdf.xacro (robot description, xacro)
@@ -56,15 +56,9 @@
 		<origin xyz="0.0 0.0 0.18" rpy="0.0 0.0 0.0" />
 	</joint>
-    <link name="tool0_cables_intermediate" />
-	<joint name="tool0_cables_intermediate_joint" type="fixed">
+    <link name="tool0_cables" />
+	<joint name="tool0_cables_joint" type="fixed">
 		<parent link="FT_sensor_frame" />
-		<child link = "tool0_cables_intermediate" />
+		<child link = "tool0_cables" />
 		<origin xyz="0.0 0.0 0.14" rpy="0.0 3.1416 0.0" />
 	</joint>
-    <link name="tool0_cables" />
-	<joint name="tool0_cables_joint" type="fixed">
-		<parent link="tool0_cables_intermediate" />
-		<child link = "tool0_cables" />
-		<origin xyz="0.0 0.0 0.0" rpy="0.0 0.0 -0.785398" />
-	</joint>
 </robot>

Commit message: Reduced all joint limits for safety

File: robot_models/urdf_models/robot_setups/robelix/use_case_setup_robelix_fixed.urdf (robot description, URDF)
Before this commit: robot robelix_neura_robot, 37 links, 36 joints
Joints:
- joint maira7M_joint1: limit lower=-3.14159 upper=3.14159 effort=432 velocity=2.0944 -> lower=-3.14159 upper=3.14159 effort=432 velocity=1.0472
- joint maira7M_joint2: limit lower=-2.0944 upper=2.0944 effort=432 velocity=2.0944 -> lower=-2.0944 upper=2.0944 effort=432 velocity=1.0472
- joint maira7M_joint3: limit lower=-3.14159 upper=3.14159 effort=217 velocity=2.618 -> lower=-3.14159 upper=3.14159 effort=217 velocity=1.0472
- joint maira7M_joint4: limit lower=-2.618 upper=2.618 effort=217 velocity=2.618 -> lower=-2.618 upper=2.618 effort=217 velocity=1.0472
- joint maira7M_joint5: limit lower=-3.14159 upper=3.14159 effort=57 velocity=3.8397 -> lower=-3.14159 upper=3.14159 effort=57 velocity=1.0472
- joint maira7M_joint6: limit lower=-3.14159 upper=3.14159 effort=57 velocity=3.8397 -> lower=-3.14159 upper=3.14159 effort=57 velocity=1.0472

File: robot_models/urdf_models/robot_setups/robelix/use_case_setup_robelix_mobile.urdf (robot description, URDF)
Before this commit: robot robelix_neura_robot, 39 links, 38 joints
Joints:
- joint maira7M_joint1: limit lower=-3.14159 upper=3.14159 effort=432 velocity=2.0944 -> lower=-3.14159 upper=3.14159 effort=432 velocity=1.0472
- joint maira7M_joint2: limit lower=-2.0944 upper=2.0944 effort=432 velocity=2.0944 -> lower=-2.0944 upper=2.0944 effort=432 velocity=1.0472
- joint maira7M_joint3: limit lower=-3.14159 upper=3.14159 effort=217 velocity=2.618 -> lower=-3.14159 upper=3.14159 effort=217 velocity=1.0472
- joint maira7M_joint4: limit lower=-2.618 upper=2.618 effort=217 velocity=2.618 -> lower=-2.618 upper=2.618 effort=217 velocity=1.0472
- joint maira7M_joint5: limit lower=-3.14159 upper=3.14159 effort=57 velocity=3.8397 -> lower=-3.14159 upper=3.14159 effort=57 velocity=1.0472
- joint maira7M_joint6: limit lower=-3.14159 upper=3.14159 effort=57 velocity=3.8397 -> lower=-3.14159 upper=3.14159 effort=57 velocity=1.0472

Commit message: One peg insertion working

File: robot_models/urdf_models/robot_setups/robelix/use_case_setup_robelix_fixed.urdf (robot description, URDF)
Before this commit: robot robelix_neura_robot, 37 links, 36 joints
Links:
- added link tool0_grip_rot
- added link tool0_insertions
Joints:
- added joint tool0_grip_rot_joint: type fixed, parent tool0_grip, child tool0_grip_rot, origin xyz=0.0 0.0 0.0 rpy=0.0 -1.0472 0.0
- added joint tool0_insertions_joint: type fixed, parent tool0_grip_rot, child tool0_insertions, origin xyz=0.0 0.0 -0.085 rpy=0.0 0.0 -1.5708
- joint tool0_grip_joint: origin xyz=0.0 0.0 0.18 rpy=0.0 0.0 0.0 -> xyz=0.0 0.0 0.18 rpy=0.0 3.1416 0.0

File: robot_models/urdf_models/robot_setups/robelix/use_case_setup_robelix_fixed.urdf.xacro (robot description, xacro)
@@ -25,5 +25,17 @@
 		<parent link="FT_sensor_frame" />
 		<child link = "tool0_grip" />
-		<origin xyz="0.0 0.0 0.18" rpy="0.0 0.0 0.0" />
+		<origin xyz="0.0 0.0 0.18" rpy="0.0 3.1416 0.0" />
+	</joint>
+	<link name="tool0_grip_rot" />
+	<joint name="tool0_grip_rot_joint" type="fixed">
+		<parent link="tool0_grip" />
+		<child link = "tool0_grip_rot" />
+		<origin xyz="0.0 0.0 0.0" rpy="0.0 -1.0472 0.0" />
+	</joint>
+	<link name="tool0_insertions" />
+	<joint name="tool0_insertions_joint" type="fixed">
+		<parent link="tool0_grip_rot" />
+		<child link = "tool0_insertions" />
+		<origin xyz="0.0 0.0 -0.085" rpy="0.0 0.0 -1.5708" />
 	</joint>
     <link name="tool0_cables" />

File: robot_models/urdf_models/robot_setups/robelix/use_case_setup_robelix_mobile.urdf (robot description, URDF)
Before this commit: robot robelix_neura_robot, 39 links, 38 joints
Joints:
- joint tool0_grip_joint: origin xyz=0.0 0.0 0.18 rpy=0.0 0.0 0.0 -> xyz=0.0 0.0 0.18 rpy=0.0 3.1416 0.0

File: robot_models/urdf_models/robot_setups/robelix/use_case_setup_robelix_mobile.urdf.xacro (robot description, xacro)
@@ -54,5 +54,5 @@
 		<parent link="FT_sensor_frame" />
 		<child link = "tool0_grip" />
-		<origin xyz="0.0 0.0 0.18" rpy="0.0 0.0 0.0" />
+		<origin xyz="0.0 0.0 0.18" rpy="0.0 3.1416 0.0" />
 	</joint>
     <link name="tool0_cables" />

Commit message: Working before demo, more testing needed. FSM generation fast

File: robot_models/urdf_models/robot_setups/robelix/use_case_setup_robelix_fixed.urdf (robot description, URDF)
Before this commit: robot robelix_neura_robot, 39 links, 38 joints
Joints:
- joint tool0_cables_joint: origin xyz=0.0 0.0 0.14 rpy=0.0 3.1416 0.0 -> xyz=0.0 0.0 0.132 rpy=0.0 3.1416 0.0
- joint tool0_grip_joint: origin xyz=0.0 0.0 0.18 rpy=0.0 3.1416 0.0 -> xyz=0.0 0.0 0.172 rpy=0.0 3.1416 0.0

File: robot_models/urdf_models/robot_setups/robelix/use_case_setup_robelix_fixed.urdf.xacro (robot description, xacro)
@@ -25,5 +25,5 @@
 		<parent link="FT_sensor_frame" />
 		<child link = "tool0_grip" />
-		<origin xyz="0.0 0.0 0.18" rpy="0.0 3.1416 0.0" />
+		<origin xyz="0.0 0.0 0.172" rpy="0.0 3.1416 0.0" />
 	</joint>
 	<link name="tool0_grip_rot" />
@@ -43,5 +43,5 @@
 		<parent link="FT_sensor_frame" />
 		<child link = "tool0_cables" />
-		<origin xyz="0.0 0.0 0.14" rpy="0.0 3.1416 0.0" />
+		<origin xyz="0.0 0.0 0.132" rpy="0.0 3.1416 0.0" />
 	</joint>
 </robot>

File: robot_models/urdf_models/robot_setups/robelix/use_case_setup_robelix_mobile.urdf (robot description, URDF)
Before this commit: robot robelix_neura_robot, 41 links, 40 joints
Joints:
- joint tool0_cables_joint: origin xyz=0.0 0.0 0.14 rpy=0.0 3.1416 0.0 -> xyz=0.0 0.0 0.132 rpy=0.0 3.1416 0.0
- joint tool0_grip_joint: origin xyz=0.0 0.0 0.18 rpy=0.0 3.1416 0.0 -> xyz=0.0 0.0 0.172 rpy=0.0 3.1416 0.0

File: robot_models/urdf_models/robot_setups/robelix/use_case_setup_robelix_mobile.urdf.xacro (robot description, xacro)
@@ -54,5 +54,5 @@
 		<parent link="FT_sensor_frame" />
 		<child link = "tool0_grip" />
-		<origin xyz="0.0 0.0 0.18" rpy="0.0 3.1416 0.0" />
+		<origin xyz="0.0 0.0 0.172" rpy="0.0 3.1416 0.0" />
 	</joint>
     <link name="tool0_grip_rot" />
@@ -72,5 +72,5 @@
 		<parent link="FT_sensor_frame" />
 		<child link = "tool0_cables" />
-		<origin xyz="0.0 0.0 0.14" rpy="0.0 3.1416 0.0" />
+		<origin xyz="0.0 0.0 0.132" rpy="0.0 3.1416 0.0" />
 	</joint>
 </robot>
