Commit message: Last version working before sending the robot to the fair

File: robot_models/urdf_models/robot_setups/robelix/use_case_setup_robelix_fixed.urdf (robot description, URDF)
Before this commit: robot robelix_neura_robot, 39 links, 38 joints
Joints:
- joint tool0_cables_joint: origin xyz=0.0 0.0 0.132 rpy=0.0 3.1416 0.0 -> xyz=0.0 0.0 0.14 rpy=0.0 3.1416 0.0
- joint tool0_grip_joint: origin xyz=0.0 0.0 0.172 rpy=0.0 3.1416 0.0 -> xyz=0.0 0.0 0.18 rpy=0.0 3.1416 0.0

File: robot_models/urdf_models/robot_setups/robelix/use_case_setup_robelix_fixed.urdf.xacro (robot description, xacro)
@@ -25,5 +25,5 @@
 		<parent link="FT_sensor_frame" />
 		<child link = "tool0_grip" />
-		<origin xyz="0.0 0.0 0.172" rpy="0.0 3.1416 0.0" />
+		<origin xyz="0.0 0.0 0.18" rpy="0.0 3.1416 0.0" />
 	</joint>
 	<link name="tool0_grip_rot" />
@@ -43,5 +43,5 @@
 		<parent link="FT_sensor_frame" />
 		<child link = "tool0_cables" />
-		<origin xyz="0.0 0.0 0.132" rpy="0.0 3.1416 0.0" />
+		<origin xyz="0.0 0.0 0.14" rpy="0.0 3.1416 0.0" />
 	</joint>
 </robot>

File: robot_models/urdf_models/robot_setups/robelix/use_case_setup_robelix_mobile.urdf (robot description, URDF)
Before this commit: robot robelix_neura_robot, 41 links, 40 joints
Joints:
- joint tool0_cables_joint: origin xyz=0.0 0.0 0.132 rpy=0.0 3.1416 0.0 -> xyz=0.0 0.0 0.14 rpy=0.0 3.1416 0.0
- joint tool0_grip_joint: origin xyz=0.0 0.0 0.172 rpy=0.0 3.1416 0.0 -> xyz=0.0 0.0 0.18 rpy=0.0 3.1416 0.0

File: robot_models/urdf_models/robot_setups/robelix/use_case_setup_robelix_mobile.urdf.xacro (robot description, xacro)
@@ -54,5 +54,5 @@
 		<parent link="FT_sensor_frame" />
 		<child link = "tool0_grip" />
-		<origin xyz="0.0 0.0 0.172" rpy="0.0 3.1416 0.0" />
+		<origin xyz="0.0 0.0 0.18" rpy="0.0 3.1416 0.0" />
 	</joint>
     <link name="tool0_grip_rot" />
@@ -72,5 +72,5 @@
 		<parent link="FT_sensor_frame" />
 		<child link = "tool0_cables" />
-		<origin xyz="0.0 0.0 0.132" rpy="0.0 3.1416 0.0" />
+		<origin xyz="0.0 0.0 0.14" rpy="0.0 3.1416 0.0" />
 	</joint>
 </robot>
