Commit message: Deleted unnecesary files and minor fixes

File: robot_models/urdf_models/robot_setups/ur10/robot_tools.urdf.xacro (robot description, xacro)
@@ -23,5 +23,5 @@
     <visual>
       <geometry>
-        <mesh filename="package://etasl_ros2_application_template/robot_description/meshes/adaptor.stl" scale=".001 .001 .001"/>
+        <mesh filename="package://etasl_ros2_application_template/robot_models/urdf_models/meshes/adaptor.stl" scale=".001 .001 .001"/>
       </geometry>
       <material name="Dark_Grey">
@@ -31,5 +31,5 @@
     <collision>
       <geometry>
-        <mesh filename="package://etasl_ros2_application_template/robot_description/meshes/adaptor.stl" scale=".001 .001 .001"/>
+        <mesh filename="package://etasl_ros2_application_template/robot_models/urdf_models/meshes/adaptor.stl" scale=".001 .001 .001"/>
       </geometry>
     </collision>
@@ -44,5 +44,5 @@
     <visual>
       <geometry>
-        <mesh filename="package://etasl_ros2_application_template/robot_description/meshes/load_cell_67.stl" scale=".001 .001 .001"/>
+        <mesh filename="package://etasl_ros2_application_template/robot_models/urdf_models/meshes/load_cell_67.stl" scale=".001 .001 .001"/>
       </geometry>
       <material name="Blue">
@@ -52,5 +52,5 @@
     <collision>
       <geometry>
-        <mesh filename="package://etasl_ros2_application_template/robot_description/meshes/load_cell_67.stl" scale=".001 .001 .001"/>
+        <mesh filename="package://etasl_ros2_application_template/robot_models/urdf_models/meshes/load_cell_67.stl" scale=".001 .001 .001"/>
       </geometry>
     </collision>

Commit message: Added headers to all code files and cleaned repo. Also fixes given the new name

File: robot_models/urdf_models/robot_setups/ur10/robot_tools.urdf.xacro (robot description, xacro)
@@ -23,5 +23,5 @@
     <visual>
       <geometry>
-        <mesh filename="package://etasl_ros2_application_template/robot_models/urdf_models/meshes/adaptor.stl" scale=".001 .001 .001"/>
+        <mesh filename="package://crospi_application_template/robot_models/urdf_models/meshes/adaptor.stl" scale=".001 .001 .001"/>
       </geometry>
       <material name="Dark_Grey">
@@ -31,5 +31,5 @@
     <collision>
       <geometry>
-        <mesh filename="package://etasl_ros2_application_template/robot_models/urdf_models/meshes/adaptor.stl" scale=".001 .001 .001"/>
+        <mesh filename="package://crospi_application_template/robot_models/urdf_models/meshes/adaptor.stl" scale=".001 .001 .001"/>
       </geometry>
     </collision>
@@ -44,5 +44,5 @@
     <visual>
       <geometry>
-        <mesh filename="package://etasl_ros2_application_template/robot_models/urdf_models/meshes/load_cell_67.stl" scale=".001 .001 .001"/>
+        <mesh filename="package://crospi_application_template/robot_models/urdf_models/meshes/load_cell_67.stl" scale=".001 .001 .001"/>
       </geometry>
       <material name="Blue">
@@ -52,5 +52,5 @@
     <collision>
       <geometry>
-        <mesh filename="package://etasl_ros2_application_template/robot_models/urdf_models/meshes/load_cell_67.stl" scale=".001 .001 .001"/>
+        <mesh filename="package://crospi_application_template/robot_models/urdf_models/meshes/load_cell_67.stl" scale=".001 .001 .001"/>
       </geometry>
     </collision>

File: robot_models/urdf_models/robot_setups/ur10/use_case_setup_ur10.urdf (robot description, URDF)
Before this commit: robot etasl_vision_scene, 15 links, 14 joints
Links:
- link adaptor_link: geometry collision mesh filename=package://crospi_application_template/robot_models/urdf_mod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 scale=.001 .001 .001; visual mesh filename=package://crospi_application_template/robot_models/urdf_mod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 scale=.001 .001 .001
- link load_cell_link: geometry collision mesh filename=package://crospi_application_template/robot_models/urdf_mod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 scale=.001 .001 .001; visual mesh filename=package://crospi_application_template/robot_models/urdf_mod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 scale=.001 .001 .001

File: robot_models/urdf_models/robot_setups/ur10/use_case_setup_ur10.urdf.xacro (robot description, xacro)
@@ -2,7 +2,7 @@
 <robot xmlns:xacro="http://www.ros.org/wiki/xacro" name="etasl_vision_scene" >
 	<!-- robot -->
-	<xacro:include filename="$(find etasl_ros2_application_template)/robot_models/urdf_models/robot_setups/ur10/robot_tools.urdf.xacro"/>
+	<xacro:include filename="$(find crospi_application_template)/robot_models/urdf_models/robot_setups/ur10/robot_tools.urdf.xacro"/>
 	<!-- environment -->
-	<xacro:include filename="$(find etasl_ros2_application_template)/robot_models/urdf_models/robot_setups/ur10/environment.urdf.xacro"/>
+	<xacro:include filename="$(find crospi_application_template)/robot_models/urdf_models/robot_setups/ur10/environment.urdf.xacro"/>
 	<xacro:property name="pi" value="3.14159265" />
 	<xacro:property name="x_w" value="0"/>

File: robot_models/urdf_models/robot_setups/ur10e/use_case_setup_ur10e.urdf.xacro (robot description, xacro)
@@ -17,5 +17,5 @@
 	</xacro:ur_robot>
 	<!-- environment
-	<xacro:include filename="$(find etasl_ros2_application_template)/robot_models/urdf_models/robot_setups/ur10e/environment.urdf.xacro"/>
+	<xacro:include filename="$(find crospi_application_template)/robot_models/urdf_models/robot_setups/ur10e/environment.urdf.xacro"/>
 	<xacro:property name="pi" value="3.14159265" />
 	<xacro:property name="x_w" value="0"/>
